File: flight-computer.sch (KiCad schematic (older format))
At the start: 47 parts, among them J1 Throttle/BEC, J2 Servo 1, J3 Servo 2, J4 Servo 3, J5 Servo 4, J6 Breakout, J7 External Power, J8 Ext, SW1 SW_Push, U1 TMP102, U2 BNO080, U3 MPL3115A2, U4 TEENSY36, Y1 32.768kHz

Commit message: New teensy footprint
Parts:
- C1, C10, C11, C2, C3, C5, C6, C7, C8, C9: footprint (none) -> Capacitor_SMD:C_0402_1005Metric
- D1, D2: footprint (none) -> Diode_SMD:D_SOD-123F
- D3, D4: footprint (none) -> LED_SMD:LED_0603_1608Metric
- J1, J2, J3, J4, J5, J8: footprint (none) -> Connector_PinSocket_2.54mm:PinSocket_1x03_P2.54mm_Vertical
- J6: footprint (none) -> Connector_PinSocket_2.54mm:PinSocket_1x08_P2.54mm_Vertical
- J7: footprint (none) -> Connector_PinSocket_2.54mm:PinSocket_1x02_P2.54mm_Vertical
- R1, R10, R11, R12, R13, R14, R15, R16, R17, R18, R2, R3, R4, R5, R6, R7, R8, R9: footprint (none) -> Resistor_SMD:R_0402_1005Metric
- SW1: footprint (none) -> Button_Switch_SMD:SW_SPST_PTS810
- U4: footprint (none) -> flight-computer:TEENSY36
- Y1: footprint (none) -> Crystal:Crystal_SMD_3215-2Pin_3.2x1.5mm
Connections:
- net D2: now also J6.6 (Pin_6); no longer J6.8 (Pin_8)
- net SCL2: now also J6.8 (Pin_8); no longer J6.7 (Pin_7)
- net SDA2: now also J6.7 (Pin_7); no longer J6.6 (Pin_6)

Commit message: Laying out PCB
Parts:
- removed J6: Breakout, Connector_PinSocket_2.54mm:PinSocket_1x08_P2.54mm_Vertical, symbol Connector_Generic:Conn_01x08
- removed J7: External Power, Connector_PinSocket_2.54mm:PinSocket_1x02_P2.54mm_Vertical, symbol Connector_Generic:Conn_01x02
- added D3: GREEN, LED_SMD:LED_0603_1608Metric, symbol Device:LED
- added J6: Breakout1, Connector_PinSocket_2.54mm:PinSocket_1x08_P2.54mm_Vertical, symbol Connector_Generic:Conn_01x07
- added J7: Power, Connector_PinSocket_2.54mm:PinSocket_1x05_P2.54mm_Vertical, symbol Connector_Generic:Conn_01x05
- added J9: Breakout2, Connector_PinSocket_2.54mm:PinSocket_1x08_P2.54mm_Vertical, symbol Connector_Generic:Conn_01x07
- added R17: 2k, Resistor_SMD:R_0402_1005Metric, symbol Device:R_Small
- C4: footprint (none) -> Capacitor_SMD:C_0402_1005Metric
- renumbered D3 to D4, D4 to D5, R17 to R18, R18 to R19
Connections:
- net +3V3: now also J7.3 (Pin_3), R17.2
- net GND: now also D3.1 (K), J7.4 (Pin_4)
- net RX1: now also J6.4 (Pin_4)
- net SCL2: now also J6.7 (Pin_7)
- net SDA2: now also J6.6 (Pin_6)
- net TX1: now also J6.5 (Pin_5)
- net VEXT: now also J7.2 (Pin_2)
- net VIN: now also J7.1 (Pin_1)
- net D26: now reaches U4.18 (D26)
- net D26: now also J6.1 (Pin_1)
- net D27: now reaches U4.19 (D27)
- net D27: now also J9.1 (Pin_1)
- net D31: now reaches U4.23 (D31_A12)
- net D31: now also J6.2 (Pin_2)
- net D32: now reaches U4.24 (D32_A13)
- net D32: now also J6.3 (Pin_3)
- net GNDA: now reaches U4.26 (AGND)
- net GNDA: now also J7.5 (Pin_5)
- net DAC1: now reaches U4.40 (A22)
- net DAC1: now also J9.3 (Pin_3)
- net DAC0: now reaches U4.41 (A21)
- net DAC0: now also J9.2 (Pin_2)
- net D36: now reaches U4.45 (D36_A17)
- net D36: now also J9.4 (Pin_4)
- net D35: now reaches U4.46 (D35_A16)
- net D35: now also J9.5 (Pin_5)
- net RX5: now reaches U4.47 (D34_A15)
- net RX5: now also J9.6 (Pin_6)
- net TX5: now reaches U4.48 (D33_A14)
- net TX5: now also J9.7 (Pin_7)
- net D2: no longer names the net of U4.4 (D2)
- new net: D3.2 (A), R17.1
- no-connect marks 22 -> 12
Other:
- note added: "Power LED"
- moved on the sheet: C1, C5, D4, D5, R1, R11, R18, R19, R2, R3, R4, SW1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

Commit message: New crystal footprint, layout changes
Parts:
- J1, J2, J3, J4, J5, J8: footprint Connector_PinSocket_2.54mm:PinSocket_1x03_P2.54mm_Vertical -> Connector_PinHeader_2.54mm:PinHeader_1x03_P2.54mm_Vertical
- J6, J9: footprint Connector_PinSocket_2.54mm:PinSocket_1x08_P2.54mm_Vertical -> Connector_PinHeader_2.54mm:PinHeader_1x07_P2.54mm_Vertical
- J7: footprint Connector_PinSocket_2.54mm:PinSocket_1x05_P2.54mm_Vertical -> Connector_PinHeader_2.54mm:PinHeader_1x05_P2.54mm_Vertical
- U1: MPN (none) -> TMP102AIDRLR
- U2: MPN (none) -> BNO080
- U3: MPN (none) -> MPL3115A2
- Y1: footprint Crystal:Crystal_SMD_3215-2Pin_3.2x1.5mm -> flight-computer:ABS07; MPN (none) -> ABS07-32.768KHZ-1-T
Changed lines of the file:
@@
 F 2 "Package_LGA:LGA-8_3x5mm_P1.25mm" H 5550 1600 50  0001 C CNN
 F 3 "" H 5550 1600 50  0001 C CNN
+F 4 "MPL3115A2" H 5550 1600 50  0001 C CNN "MPN"
 	1    5550 1600
 	1    0    0    -1
@@
 F 0 "J1" H 1580 4592 50  0000 L CNN
 F 1 "Throttle/BEC" H 1580 4501 50  0000 L CNN
-F 2 "Connector_PinSocket_2.54mm:PinSocket_1x03_P2.54mm_Vertical" H 1500 4550 50  0001 C CNN
+F 2 "Connector_PinHeader_2.54mm:PinHeader_1x03_P2.54mm_Vertical" H 1500 4550 50  0001 C CNN
 F 3 "~" H 1500 4550 50  0001 C CNN
 	1    1500 4550
@@
 F 0 "J2" H 1580 4942 50  0000 L CNN
 F 1 "Servo 1" H 1580 4851 50  0000 L CNN
-F 2 "Connector_PinSocket_2.54mm:PinSocket_1x03_P2.54mm_Vertical" H 1500 4900 50  0001 C CNN
+F 2 "Connector_PinHeader_2.54mm:PinHeader_1x03_P2.54mm_Vertical" H 1500 4900 50  0001 C CNN
 F 3 "~" H 1500 4900 50  0001 C CNN
 	1    1500 4900
@@
 F 0 "J3" H 1580 5292 50  0000 L CNN
 F 1 "Servo 2" H 1580 5201 50  0000 L CNN
-F 2 "Connector_PinSocket_2.54mm:PinSocket_1x03_P2.54mm_Vertical" H 1500 5250 50  0001 C CNN
+F 2 "Connector_PinHeader_2.54mm:PinHeader_1x03_P2.54mm_Vertical" H 1500 5250 50  0001 C CNN
 F 3 "~" H 1500 5250 50  0001 C CNN
 	1    1500 5250
@@
 F 0 "J4" H 1580 5642 50  0000 L CNN
 F 1 "Servo 3" H 1580 5551 50  0000 L CNN
-F 2 "Connector_PinSocket_2.54mm:PinSocket_1x03_P2.54mm_Vertical" H 1500 5600 50  0001 C CNN
+F 2 "Connector_PinHeader_2.54mm:PinHeader_1x03_P2.54mm_Vertical" H 1500 5600 50  0001 C CNN
 F 3 "~" H 1500 5600 50  0001 C CNN
 	1    1500 5600
@@
 F 0 "J5" H 1580 5992 50  0000 L CNN
 F 1 "Servo 4" H 1580 5901 50  0000 L CNN
-F 2 "Connector_PinSocket_2.54mm:PinSocket_1x03_P2.54mm_Vertical" H 1500 5950 50  0001 C CNN
+F 2 "Connector_PinHeader_2.54mm:PinHeader_1x03_P2.54mm_Vertical" H 1500 5950 50  0001 C CNN
 F 3 "~" H 1500 5950 50  0001 C CNN
 	1    1500 5950
@@
 F 2 "Package_TO_SOT_SMD:SOT-563" H 1450 2700 50  0001 C CNN
 F 3 "" H 1450 2700 50  0001 C CNN
+F 4 "TMP102AIDRLR" H 1750 2700 50  0001 C CNN "MPN"
 	1    1750 2700
 	1    0    0    -1
@@
 F 0 "J8" H 2730 5992 50  0000 L CNN
 F 1 "Ext" H 2730 5901 50  0000 L CNN
-F 2 "Connector_PinSocket_2.54mm:PinSocket_1x03_P2.54mm_Vertical" H 2650 5950 50  0001 C CNN
+F 2 "Connector_PinHeader_2.54mm:PinHeader_1x03_P2.54mm_Vertical" H 2650 5950 50  0001 C CNN
 F 3 "~" H 2650 5950 50  0001 C CNN
 	1    2650 5950
@@
 F 2 "Package_LGA:LGA-28_5.2x3.8mm_P0.5mm" H 4900 2950 50  0001 C CNN
 F 3 "" H 4900 2950 50  0001 C CNN
+F 4 "BNO080" H 4900 2950 50  0001 C CNN "MPN"
 	1    4900 2950
 	1    0    0    -1
@@
 F 0 "Y1" V 5650 3900 50  0000 L CNN
 F 1 "32.768kHz" V 5750 3900 50  0000 L CNN
-F 2 "Crystal:Crystal_SMD_3215-2Pin_3.2x1.5mm" H 5700 3800 50  0001 C CNN
+F 2 "flight-computer:ABS07" H 5700 3800 50  0001 C CNN
 F 3 "~" H 5700 3800 50  0001 C CNN
+F 4 "ABS07-32.768KHZ-1-T" V 5700 3800 50  0001 C CNN "MPN"
 	1    5700 3800
 	0    1    1    0
@@
 F 0 "J7" H 2730 5542 50  0000 L CNN
 F 1 "Power" H 2730 5451 50  0000 L CNN
-F 2 "Connector_PinSocket_2.54mm:PinSocket_1x05_P2.54mm_Vertical" H 2650 5500 50  0001 C CNN
+F 2 "Connector_PinHeader_2.54mm:PinHeader_1x05_P2.54mm_Vertical" H 2650 5500 50  0001 C CNN
 F 3 "~" H 2650 5500 50  0001 C CNN
 	1    2650 5500
@@
 F 0 "J6" H 2730 4892 50  0000 L CNN
 F 1 "Breakout1" H 2730 4801 50  0000 L CNN
-F 2 "Connector_PinSocket_2.54mm:PinSocket_1x08_P2.54mm_Vertical" H 2650 4850 50  0001 C CNN
+F 2 "Connector_PinHeader_2.54mm:PinHeader_1x07_P2.54mm_Vertical" H 2650 4850 50  0001 C CNN
 F 3 "~" H 2650 4850 50  0001 C CNN
 	1    2650 4850
@@
 F 0 "J9" H 3930 5392 50  0000 L CNN
 F 1 "Breakout2" H 3930 5301 50  0000 L CNN
-F 2 "Connector_PinSocket_2.54mm:PinSocket_1x08_P2.54mm_Vertical" H 3850 5350 50  0001 C CNN
+F 2 "Connector_PinHeader_2.54mm:PinHeader_1x07_P2.54mm_Vertical" H 3850 5350 50  0001 C CNN
 F 3 "~" H 3850 5350 50  0001 C CNN
 	1    3850 5350
