File: flight-computer.sch (KiCad schematic (older format))
At the start: 50 parts, among them J1 Throttle/BEC, J2 Servo 1, J3 Servo 2, J4 Servo 3, J5 Servo 4, J6 Breakout1, J7 Power, J8 Ext, J9 Breakout2, SW1 SW_Push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

Commit message: Routing
Parts:
- removed D1: SS14FL, Diode_SMD:D_SOD-123F, symbol Device:D_Schottky_Small_ALT
- renumbered D2 to D1, D3 to D2, D4 to D3, D5 to D4
Connections:
- net VEXT is gone; now on net VBEC: J7.2 (Pin_2)
Other:
- moved on the sheet: D1
Changed lines of the file:
@@
 	1    0    0    -1
 $EndComp
-Text Label 2400 1250 2    50   ~ 0
+Text Label 2000 1300 2    50   ~ 0
 VIN
-Text Label 1450 1400 0    50   ~ 0
+Text Label 1450 1300 0    50   ~ 0
 VBEC
 Wire Wire Line
@@
 VBEC
 $Comp
-L Device:D_Schottky_Small_ALT D2
+L Device:D_Schottky_Small_ALT D1
 U 1 1 5E4B50E3
-P 1800 1400
-F 0 "D2" H 1800 1600 50  0000 C CNN
-F 1 "SS14FL" H 1900 1500 50  0000 C CNN
-F 2 "Diode_SMD:D_SOD-123F" V 1800 1400 50  0001 C CNN
-F 3 "~" V 1800 1400 50  0001 C CNN
-	1    1800 1400
+P 1750 1300
+F 0 "D1" H 1750 1500 50  0000 C CNN
+F 1 "SS14FL" H 1850 1400 50  0000 C CNN
+F 2 "Diode_SMD:D_SOD-123F" V 1750 1300 50  0001 C CNN
+F 3 "~" V 1750 1300 50  0001 C CNN
+	1    1750 1300
 	-1   0    0    1
 $EndComp
@@
 $EndComp
 $Comp
-L Device:LED D5
+L Device:LED D4
 U 1 1 5E5B9117
 P 8150 4900
-F 0 "D5" H 8150 5050 50  0000 C CNN
+F 0 "D4" H 8150 5050 50  0000 C CNN
 F 1 "BLUE" H 8150 5150 50  0000 C CNN
 F 2 "LED_SMD:LED_0603_1608Metric" H 8150 4900 50  0001 C CNN
@@
 $EndComp
 $Comp
-L Device:LED D4
+L Device:LED D3
 U 1 1 5E5B9CB0
 P 8150 4550
-F 0 "D4" H 8150 4700 50  0000 C CNN
+F 0 "D3" H 8150 4700 50  0000 C CNN
 F 1 "RED" H 8150 4800 50  0000 C CNN
 F 2 "LED_SMD:LED_0603_1608Metric" H 8150 4550 50  0001 C CNN
@@
 Text Label 1100 5850 0    50   ~ 0
 SER4
-Wire Wire Line
-	1900 1400 2050 1400
 $Comp
 L flight-computer:TMP102 U1
@@
 	9000 3700 8900 3700
 Wire Wire Line
-	2050 1100 2050 1250
-Wire Wire Line
-	1700 1100 1450 1100
-$Comp
-L Device:D_Schottky_Small_ALT D1
-U 1 1 5E6430D3
-P 1800 1100
-F 0 "D1" H 1800 1300 50  0000 C CNN
-F 1 "SS14FL" H 1900 1200 50  0000 C CNN
-F 2 "Diode_SMD:D_SOD-123F" V 1800 1100 50  0001 C CNN
-F 3 "~" V 1800 1100 50  0001 C CNN
-	1    1800 1100
-	-1   0    0    1
-$EndComp
-Text Label 1450 1100 0    50   ~ 0
-VEXT
-Wire Wire Line
-	2050 1100 1900 1100
-Wire Wire Line
 	7900 3900 7750 3900
 Text Label 7750 3900 0    50   ~ 0
@@
 Text Notes 7900 1050 0    50   ~ 0
 Teensy 3.6 Microcontroller
-Wire Wire Line
-	2050 1250 2400 1250
-Connection ~ 2050 1250
-Wire Wire Line
-	2050 1250 2050 1400
 $Comp
 L power:+3V3 #PWR034
@@
 $EndComp
 Text Label 2300 5400 0    50   ~ 0
-VEXT
+VBEC
 Wire Wire Line
 	2450 5400 2300 5400
@@
 	1    0    0    -1
 $EndComp
-Text Notes 1500 950  0    50   ~ 0
+Text Notes 1500 1150 0    50   ~ 0
 Power Input
 Text Notes 5250 1150 0    50   ~ 0
@@
 NoConn ~ 8900 1500
 Wire Wire Line
-	1700 1400 1450 1400
+	1650 1300 1450 1300
 Wire Wire Line
 	4350 1950 4750 1950
@@
 $EndComp
 $Comp
-L Device:LED D3
+L Device:LED D2
 U 1 1 5E6E20C4
 P 6800 4750
-F 0 "D3" H 6800 4900 50  0000 C CNN
+F 0 "D2" H 6800 4900 50  0000 C CNN
 F 1 "GREEN" H 6800 5000 50  0000 C CNN
 F 2 "LED_SMD:LED_0603_1608Metric" H 6800 4750 50  0001 C CNN
@@
 Text Label 2150 4550 0    50   ~ 0
 D26
+Wire Wire Line
+	1850 1300 2000 1300
 $EndSCHEMATC

Commit message: Fixed C4 footprint
Parts:
- C4: footprint Capacitor_SMD:C_0402_1005Metric -> Capacitor_SMD:C_1206_3216Metric
Changed lines of the file:
@@
 F 0 "C4" H 4150 1900 50  0000 L CNN
 F 1 "10uF" H 4050 1800 50  0000 L CNN
-F 2 "Capacitor_SMD:C_0402_1005Metric" H 4350 1850 50  0001 C CNN
+F 2 "Capacitor_SMD:C_1206_3216Metric" H 4350 1850 50  0001 C CNN
 F 3 "~" H 4350 1850 50  0001 C CNN
 	1    4350 1850

Commit message: Version 1
Parts:
- SW1: MPN (none) -> PTS810 SJM 250 SMTR LFS
Changed lines of the file:
@@
 Wire Wire Line
 	4750 1950 5100 1950
-$Comp
-L power:GND #PWR023
-U 1 1 5E6BC8C6
-P 4750 1950
-F 0 "#PWR023" H 4750 1700 50  0001 C CNN
-F 1 "GND" V 4755 1822 50  0000 R CNN
-F 2 "" H 4750 1950 50  0001 C CNN
-F 3 "" H 4750 1950 50  0001 C CNN
-	1    4750 1950
-	1    0    0    -1
-$EndComp
 Text Notes 1500 1150 0    50   ~ 0
 Power Input
@@
 P 5950 3000
 F 0 "#PWR028" H 5950 2850 50  0001 C CNN
-F 1 "+3V3" V 5950 3250 50  0000 C CNN
+F 1 "+3V3" H 5950 3150 50  0000 C CNN
 F 2 "" H 5950 3000 50  0001 C CNN
 F 3 "" H 5950 3000 50  0001 C CNN
@@
 F 2 "Button_Switch_SMD:SW_SPST_PTS810" H 4400 6150 50  0001 C CNN
 F 3 "~" H 4400 6150 50  0001 C CNN
+F 4 "PTS810 SJM 250 SMTR LFS" H 4400 5950 50  0001 C CNN "MPN"
 	1    4400 5950
 	1    0    0    -1
@@
 Wire Wire Line
 	1850 1300 2000 1300
+$Comp
+L power:GND #PWR023
+U 1 1 5E6BC8C6
+P 4750 1950
+F 0 "#PWR023" H 4750 1700 50  0001 C CNN
+F 1 "GND" V 4755 1822 50  0000 R CNN
+F 2 "" H 4750 1950 50  0001 C CNN
+F 3 "" H 4750 1950 50  0001 C CNN
+	1    4750 1950
+	1    0    0    -1
+$EndComp
 $EndSCHEMATC
